Commit message: corrected urdf

File: robot_description/hero_v3/urdf/hero_7dof_v3.urdf (robot description, URDF)
Before this commit: robot hero_7dof_v3, 14 links, 13 joints
Joints:
- joint gripper1_jaw_left_joint: origin xyz=-0.035 0.059351 0.05 rpy=1.5708 0 3.1416 -> xyz=-0.035 0.061 0.05 rpy=1.5708 0 3.1416
- joint gripper1_jaw_right_joint: origin xyz=0.035 -0.05935 0.05 rpy=-1.5708 0 3.1416 -> xyz=0.035 -0.061 0.05 rpy=-1.5708 0 3.1416

File: robot_description/hero_v3/urdf/hero_7dof_v3_rs.urdf (robot description, URDF)
Before this commit: robot hero_7dof_v3_rs, 44 links, 43 joints
Joints:
- joint gripper1_jaw_left_joint: origin xyz=-0.035 0.059351 0.05 rpy=1.5708 0 3.1416 -> xyz=-0.035 0.061 0.05 rpy=1.5708 0 3.1416
- joint gripper1_jaw_right_joint: origin xyz=0.035 -0.05935 0.05 rpy=-1.5708 0 3.1416 -> xyz=0.035 -0.061 0.05 rpy=-1.5708 0 3.1416
